File: 8085 Computer.sch (KiCad schematic (older format))
At the start: 37 parts, among them IC1 8085-8085, J1 Barrel_Jack_Switch, J2 Conn_02x20_Top_Bottom, J3 Conn_01x06_Male, SW1 SW_MEC_5E, U1 74LS00, U2 74LS00, U3 74LS244, U4 74LS245, U5 74LS373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

Commit message: Starting board layout
Parts:
- C1: footprint (none) -> Capacitor_THT:CP_Radial_Tantal_D4.5mm_P2.50mm
- C10, C11, C12, C13, C14, C4, C5, C6, C7, C8, C9: footprint (none) -> Capacitor_THT:C_Disc_D3.0mm_W2.0mm_P2.50mm
- C2, C3: footprint (none) -> Capacitor_THT:C_Disc_D3.0mm_W1.6mm_P2.50mm
- D1: footprint (none) -> Diode_THT:D_A-405_P7.62mm_Horizontal
- J1: footprint (none) -> Connector_BarrelJack:BarrelJack_Horizontal
- J2: footprint (none) -> Connector_PinHeader_2.54mm:PinHeader_2x20_P2.54mm_Vertical
- J3: footprint (none) -> Connector_PinHeader_2.54mm:PinHeader_1x06_P2.54mm_Horizontal
- R1, R2, R3, R4, R5, R6, R7, R8: footprint (none) -> Resistor_THT:R_Axial_DIN0207_L6.3mm_D2.5mm_P7.62mm_Horizontal
- SW1: footprint (none) -> Button_Switch_THT:SW_TH_Tactile_Omron_B3F-10xx
- U1: renamed from IC1; value 8085-8085 -> 8085; footprint Package_DIP:DIP-40_W25.4mm -> Package_DIP:DIP-40_W15.24mm
- U2: renamed from U3; footprint (none) -> Package_DIP:DIP-20_W7.62mm
- U3: renamed from U4; footprint (none) -> Package_DIP:DIP-20_W7.62mm
- U4: renamed from U5; footprint (none) -> Package_DIP:DIP-20_W7.62mm
- U5: renamed from U6; footprint (none) -> Package_DIP:DIP-20_W7.62mm
- U6: renamed from U7; footprint (none) -> Package_DIP:DIP-28_W15.24mm
- U8: renamed from U2; footprint (none) -> Package_DIP:DIP-16_W7.62mm
- U8: renamed from U1; footprint (none) -> Package_DIP:DIP-16_W7.62mm
- Y1: footprint (none) -> Crystal:Crystal_HC33-U_Vertical
- renumbered U8 to U7
Connections:
- no-connect marks 5 -> 6
Other:
- moved on the sheet: U8A, U8B, U8C, U8D, U8E
